File: Hardware/Selectric.sch (EAGLE design)
At the start: 57 parts, among them IC1 UDN2982SLW, IC2 UDN2982SLW, IC3 MAX3232ESE, X1 C-GRID-18-70543, X2 22-23-2041

Commit message: Modify connectors, assign I/Os
Add eC-stencil registration holes
Parts:
- removed SV1: (no value), con-lstb:MA13-2
- added R32: 1K, rcl:R-EU_M1206
- added X4: C-GRID-16-70543, con-molex:C-GRID-16-70543
- DC1: MF (none) -> TRACO; MPN (none) -> TMR1-4811
- F1: MF (none) -> Schurter; MPN (none) -> 3404.0009.11
- IC1, IC2: MF (none) -> Allegro; MPN (none) -> UDN2982SLW
- JP1, JP2: MF (none) -> WURTH; MPN (none) -> 61301611121
- JP10, JP11, JP6, JP8, JP9: MF (none) -> TE CONNECTIVITY; MPN (none) -> 826629-8
- JP5: MF (none) -> TE CONNECTIVITY; MPN (none) -> 826629-6
- JP7: MF (none) -> TE CONNECTIVITY; MPN (none) -> 826632-2
- R11: value 220R -> 1K
- X1: value C-GRID-18-70543 -> 2530-; device con-molex:C-GRID-18-70543 -> con-3m:2530-; MF (none) -> 3M; MPN (none) -> PAK100/2500-30
- X2: MF (none) -> TE CONNECTIVITY; MPN (none) -> 280371-2
- X3: MF (none) -> Amphenol; MPN (none) -> FCE17-E09PA-490
Connections:
- removed net HSD16: X1-17.S
- net D25: now also R10.2, X2-2.S
- net D26: now also X1-2.KL; no longer SV1.2
- net D27: now also X1-3.KL; no longer SV1.1
- net D28: now also X1-4.KL; no longer SV1.4
- net D29: now also X1-5.KL; no longer SV1.3
- net D30: now also X1-6.KL; no longer SV1.6
- net D31: now also X1-7.KL; no longer SV1.5
- net D32: now also X1-8.KL; no longer SV1.8
- net D33: now also X1-9.KL; no longer SV1.7
- net D34: now also X1-10.KL; no longer SV1.10
- net D35: now also X1-11.KL; no longer SV1.9
- net D36: now also X1-12.KL; no longer SV1.12
- net D37: now also X1-13.KL; no longer SV1.11
- net D38: now also X1-14.KL; no longer SV1.14
- net D39: now also X1-15.KL; no longer SV1.13
- net D40: now also X1-16.KL; no longer SV1.16
- net D41: now also X1-17.KL; no longer SV1.15
- net D42: now also X1-18.KL; no longer SV1.18
- net D43: now also X1-19.KL; no longer SV1.17
- net D44: now also X1-20.KL; no longer SV1.20
- net D45: now also X1-21.KL; no longer SV1.19
- net D46: now also X1-22.KL; no longer SV1.22
- net D47: now also X1-23.KL; no longer SV1.21
- net D48: now also X1-24.KL; no longer SV1.24
- net D49: now also X1-25.KL; no longer SV1.23
- net D50: now also X1-26.KL; no longer SV1.26
- net D51: now also X1-27.KL; no longer SV1.25
- net D52: now also R32.1, X1-28.KL; no longer R10.2, X2-2.S
- net GND: now also X1-29.KL, X1-30.KL
- net HSD1: now also X4-1.S; no longer X1-2.S
- net HSD10: now also X4-10.S; no longer X1-11.S
- net HSD11: now also X4-11.S; no longer X1-12.S
- net HSD12: now also X4-12.S; no longer X1-13.S
- net HSD13: now also X4-13.S; no longer X1-14.S
- net HSD14: now also X4-14.S; no longer X1-15.S
- net HSD15: now also X4-15.S; no longer X1-16.S
- net HSD2: now also X4-2.S; no longer X1-3.S
- net HSD3: now also X4-3.S; no longer X1-4.S
- net HSD4: now also X4-4.S; no longer X1-5.S
- net HSD5: now also X4-5.S; no longer X1-6.S
- net HSD6: now also X4-6.S; no longer X1-7.S
- net HSD7: now also X4-7.S; no longer X1-8.S
- net HSD8: now also X4-8.S; no longer X1-9.S
- net HSD9: now also X4-9.S; no longer X1-10.S
- net HSDRET: now also X4-16.S; no longer X1-18.S
- net VCC: now also R32.2
Other:
- note added: "Keyboard Inputs D38 PAR D39 T2 D40 CK D41 T1 D42 R2A D43 R1 D44 R2 D45 R5 D46 TAB D47 SP D48 BSP D49 CR D50 LF D51 UC D52 LC"
- note added: "Other Inputs D19 RXD D17 CTS D25 Switch"
- note added: "Other Outputs D18 TXD D16 RTS D53 LED"
- note added: "Printer Switch Inputs D26 C1_NC D27 CRTAB_NC D28 LC D29 C2_6_NC D30 C2_6_NO D31 CRTAB_NO D32 EOL_NC D33 EOL_NO D34 UC D35 LOCK_NC D36 LOCK_NO D37 C1_NO"
- note added: "Solenoid Outputs D2 LOCK D3 R2A D4 R1 D5 R2 D6 R5 D7 T2 D8 T1 D9 CK D10 TAB D11 SP D12 BSP D13 CR D22 INDEX D23 UC D24 LC"
- note added: "Spare I/O D0 RX0 D1 TX0 D14 D15 D20 SDA D21 SCL"
- note removed: "Keyboard Inputs D38 D39 D40 D41 D42 D43 D44 D45 D46 D47 D48 D49 D50 D51"
- note removed: "Other Inputs D0 RXD D17 CTS D52 Switch"
- note removed: "Other Outputs D1 TXD D16 RTS D53 LED"
- note removed: "Printer Switch Inputs D26 D27 D28 D29 D30 D31 D32 D33 D34 D35 D36 D37"
- note removed: "Solenoid Outputs D2 LOCK D3 D4 D5 D6 D7 D8 D9 D10 D11 D12 D22 D23 D24"

Commit message: Version as ordered
Note BoM is not necessarily accurate
Parts:
- added HSD1A: (no value), wirepad:2,15/1,0
- added R33: 1K, rcl:R-EU_M1206
- IC3: MPN (none) -> MAX3232CSE
Connections:
- net N$5 renamed HSD1A
- net D15: now also R33.1, X1-1.KL
- net HSD1: now also HSD1A.P
- net VCC: now also R33.2
